Commit message: Sep15

File: assets/botyard/panda_by_description/urdf/panda_by.urdf (robot description, URDF)
Before this commit: robot panda, 50 links, 49 joints
Links:
- link falink1: geometry visual mesh filename=package://panda_by_description/meshes/botyard/falink1.STL
- link falink2: geometry visual mesh filename=package://panda_by_description/meshes/botyard/falink2.STL
- link fallink0: geometry visual mesh filename=package://panda_by_description/meshes/botyard/fallink0.STL
- link fallink1: geometry visual mesh filename=package://panda_by_description/meshes/botyard/fallink1.STL
- link fallink2: geometry visual mesh filename=package://panda_by_description/meshes/botyard/fallink2.STL
- link farlink0: geometry visual mesh filename=package://panda_by_description/meshes/botyard/farlink0.STL
- link farlink1: geometry visual mesh filename=package://panda_by_description/meshes/botyard/farlink1.STL
- link farlink2: geometry visual mesh filename=package://panda_by_description/meshes/botyard/farlink2.STL

Commit message: “ik_Sep16_problem”

File: assets/botyard/panda_by_description/urdf/panda_by.urdf (robot description, URDF)
Before this commit: robot panda, 50 links, 49 joints
Joints:
- joint CJ0: origin xyz=0 0.02335 0.045 rpy=0 0 0 -> xyz=0 0.02335 0.045 rpy=0 -1.57 1.57
