Commit message: remove useless and add dexhand-only urdf

File: assets/botyard/ur_by_description/urdf/dexhand.urdf (robot description, URDF)
Before this commit: robot dexhand, 42 links, 41 joints
Links:
- link fabase: geometry collision mesh filename=package://ur_by_description/meshes/botyard/fabase.STL; visual mesh filename=package://ur_by_description/meshes/botyard/fabase.STL
- link falink1: geometry collision mesh filename=package://ur_by_description/meshes/botyard/falink1.STL; visual mesh filename=package://ur_by_description/meshes/botyard/falink1.STL
- link falink2: geometry collision mesh filename=package://ur_by_description/meshes/botyard/falink2.STL; visual mesh filename=package://ur_by_description/meshes/botyard/falink2.STL
- link fallink0: geometry collision mesh filename=package://ur_by_description/meshes/botyard/fallink0.STL; visual mesh filename=package://ur_by_description/meshes/botyard/fallink0.STL
- link fallink1: geometry collision mesh filename=package://ur_by_description/meshes/botyard/fallink1.STL; visual mesh filename=package://ur_by_description/meshes/botyard/fallink1.STL
- link fallink2: geometry collision mesh filename=package://ur_by_description/meshes/botyard/fallink2.STL; visual mesh filename=package://ur_by_description/meshes/botyard/fallink2.STL
- link farlink0: geometry collision mesh filename=package://ur_by_description/meshes/botyard/farlink0.STL; visual mesh filename=package://ur_by_description/meshes/botyard/farlink0.STL
- link farlink1: geometry collision mesh filename=package://ur_by_description/meshes/botyard/farlink1.STL; visual mesh filename=package://ur_by_description/meshes/botyard/farlink1.STL
- link farlink2: geometry collision mesh filename=package://ur_by_description/meshes/botyard/farlink2.STL; visual mesh filename=package://ur_by_description/meshes/botyard/farlink2.STL
- link ffbase: geometry collision mesh filename=package://ur_by_description/meshes/botyard/ffbase.STL; visual mesh filename=package://ur_by_description/meshes/botyard/ffbase.STL
- link ffdistal: geometry collision mesh filename=package://ur_by_description/meshes/botyard/ffdistal.STL; visual mesh filename=package://ur_by_description/meshes/botyard/ffdistal.STL
- link ffmiddle: geometry collision mesh filename=package://ur_by_description/meshes/botyard/ffmiddle.STL; visual mesh filename=package://ur_by_description/meshes/botyard/ffmiddle.STL
- link ffproximal: geometry collision mesh filename=package://ur_by_description/meshes/botyard/ffproximal.STL; visual mesh filename=package://ur_by_description/meshes/botyard/ffproximal.STL
- link lfbase: geometry collision mesh filename=package://ur_by_description/meshes/botyard/lfbase.STL; visual mesh filename=package://ur_by_description/meshes/botyard/lfbase.STL
- link lfdistal: geometry collision mesh filename=package://ur_by_description/meshes/botyard/lfdistal.STL; visual mesh filename=package://ur_by_description/meshes/botyard/lfdistal.STL
- link lfmiddle: geometry collision mesh filename=package://ur_by_description/meshes/botyard/lfmiddle.STL; visual mesh filename=package://ur_by_description/meshes/botyard/lfmiddle.STL
- link lfproximal: geometry collision mesh filename=package://ur_by_description/meshes/botyard/lfproximal.STL; visual mesh filename=package://ur_by_description/meshes/botyard/lfproximal.STL
- link mfbase: geometry collision mesh filename=package://ur_by_description/meshes/botyard/mfbase.STL; visual mesh filename=package://ur_by_description/meshes/botyard/mfbase.STL
- link mfdistal: geometry collision mesh filename=package://ur_by_description/meshes/botyard/mfdistal.STL; visual mesh filename=package://ur_by_description/meshes/botyard/mfdistal.STL
- link mfmiddle: geometry collision mesh filename=package://ur_by_description/meshes/botyard/mfmiddle.STL; visual mesh filename=package://ur_by_description/meshes/botyard/mfmiddle.STL
- link mfproximal: geometry collision mesh filename=package://ur_by_description/meshes/botyard/mfproximal.STL; visual mesh filename=package://ur_by_description/meshes/botyard/mfproximal.STL
- link palm: geometry collision mesh filename=package://ur_by_description/meshes/botyard/palm.STL; visual mesh filename=package://ur_by_description/meshes/botyard/palm.STL
- link pmbase: geometry collision mesh filename=package://ur_by_description/meshes/botyard/pmbase.STL; visual mesh filename=package://ur_by_description/meshes/botyard/pmbase.STL
- link rfbase: geometry collision mesh filename=package://ur_by_description/meshes/botyard/rfbase.STL; visual mesh filename=package://ur_by_description/meshes/botyard/rfbase.STL
- link rfdistal: geometry collision mesh filename=package://ur_by_description/meshes/botyard/rfdistal.STL; visual mesh filename=package://ur_by_description/meshes/botyard/rfdistal.STL
- link rfmiddle: geometry collision mesh filename=package://ur_by_description/meshes/botyard/rfmiddle.STL; visual mesh filename=package://ur_by_description/meshes/botyard/rfmiddle.STL
- link rfproximal: geometry collision mesh filename=package://ur_by_description/meshes/botyard/rfproximal.STL; visual mesh filename=package://ur_by_description/meshes/botyard/rfproximal.STL
- link thbase: geometry collision mesh filename=package://ur_by_description/meshes/botyard/thbase.STL; visual mesh filename=package://ur_by_description/meshes/botyard/thbase.STL
- link thdistal: geometry collision mesh filename=package://ur_by_description/meshes/botyard/thdistal.STL; visual mesh filename=package://ur_by_description/meshes/botyard/thdistal.STL
- link thmiddle: geometry collision mesh filename=package://ur_by_description/meshes/botyard/thmiddle.STL; visual mesh filename=package://ur_by_description/meshes/botyard/thmiddle.STL
- link thproximal: geometry collision mesh filename=package://ur_by_description/meshes/botyard/thproximal.STL; visual mesh filename=package://ur_by_description/meshes/botyard/thproximal.STL
Joints:
- joint CJ0: origin xyz=0 0.02335 0.045 rpy=0 0 0 -> xyz=0 0.02335 0.045 rpy=0 -1.57 1.57
